Commit message: CLearer urdf/xacro structure

File: alaris_gripper_description/urdf/alaris_gripper.urdf.xacro (robot description, xacro)
@@ -1,5 +1,13 @@
 <?xml version="1.0"?>
 <robot name="alaris_gripper" xmlns:xacro="http://www.ros.org/wiki/xacro">
+    <!-- Materials and Properties -->
+    <xacro:include filename="$(find alaris_gripper_description)/urdf/extras/materials.urdf.xacro"/>
+    <xacro:include filename="$(find alaris_gripper_description)/urdf/extras/properties.urdf.xacro"/>
+    <!-- Gripper Parts -->
     <xacro:include filename="$(find alaris_gripper_description)/urdf/parts/base.urdf.xacro"/>
+    <xacro:include filename="$(find alaris_gripper_description)/urdf/parts/finger.urdf.xacro"/>
     <xacro:alaris_gripper_base prefix="gripper"/>
+    <xacro:alaris_gripper_finger prefix="gripper" finger_id="1" parent="gripper_palm_link">
+        <origin xyz="0 0 0.05" rpy="0 0 0"/>
+    </xacro:alaris_gripper_finger>
 </robot>

Commit message: Added fingers

File: alaris_gripper_description/urdf/alaris_gripper.urdf.xacro (robot description, xacro)
@@ -9,5 +9,11 @@
     <xacro:alaris_gripper_base prefix="gripper"/>
     <xacro:alaris_gripper_finger prefix="gripper" finger_id="1" parent="gripper_palm_link">
-        <origin xyz="0 0 0.05" rpy="0 0 0"/>
+        <origin xyz="-0.04625 -0.0003 -0.007" rpy="0 0 -${2*PI/3}"/>
+    </xacro:alaris_gripper_finger>
+    <xacro:alaris_gripper_finger prefix="gripper" finger_id="2" parent="gripper_palm_link">
+        <origin xyz="0.0236 0.04035 -0.007" rpy="0 0 ${2*PI/3}"/>
+    </xacro:alaris_gripper_finger>
+    <xacro:alaris_gripper_finger prefix="gripper" finger_id="3" parent="gripper_palm_link">
+        <origin xyz="0.0238 -0.04035 -0.007" rpy="0 0 0"/>
     </xacro:alaris_gripper_finger>
 </robot>

Commit message: First moving parts!

File: alaris_gripper_description/urdf/alaris_gripper.urdf.xacro (robot description, xacro)
@@ -7,13 +7,13 @@
     <xacro:include filename="$(find alaris_gripper_description)/urdf/parts/base.urdf.xacro"/>
     <xacro:include filename="$(find alaris_gripper_description)/urdf/parts/finger.urdf.xacro"/>
-    <xacro:alaris_gripper_base prefix="gripper"/>
-    <xacro:alaris_gripper_finger prefix="gripper" finger_id="1" parent="gripper_palm_link">
-        <origin xyz="-0.04625 -0.0003 -0.007" rpy="0 0 -${2*PI/3}"/>
+    <xacro:alaris_gripper_base prefix="${prefix}"/>
+    <xacro:alaris_gripper_finger prefix="${prefix}" finger_id="1" parent="${prefix}_palm_link">
+        <origin xyz="-0.0435 -0.00052 -0.006" rpy="0 0 -${2*PI/3}"/>
     </xacro:alaris_gripper_finger>
-    <xacro:alaris_gripper_finger prefix="gripper" finger_id="2" parent="gripper_palm_link">
-        <origin xyz="0.0236 0.04035 -0.007" rpy="0 0 ${2*PI/3}"/>
+    <xacro:alaris_gripper_finger prefix="${prefix}" finger_id="2" parent="${prefix}_palm_link">
+        <origin xyz="0.022 0.03785 -0.006" rpy="0 0 ${2*PI/3}"/>
     </xacro:alaris_gripper_finger>
-    <xacro:alaris_gripper_finger prefix="gripper" finger_id="3" parent="gripper_palm_link">
-        <origin xyz="0.0238 -0.04035 -0.007" rpy="0 0 0"/>
+    <xacro:alaris_gripper_finger prefix="${prefix}" finger_id="3" parent="${prefix}_palm_link">
+        <origin xyz="0.0226 -0.03785 -0.006" rpy="0 0 0"/>
     </xacro:alaris_gripper_finger>
 </robot>

File: alaris_gripper_description/urdf/extras/properties.urdf.xacro (robot description, xacro)
@@ -2,3 +2,4 @@
 <robot name="gripper_materials" xmlns:xacro="http://www.ros.org/wiki/xacro">
     <xacro:property name="PI" value="3.14159"/>
+    <xacro:property name="prefix" value="gripper"/>
 </robot>

File: alaris_gripper_description/urdf/parts/base.urdf.xacro (robot description, xacro)
@@ -154,6 +154,8 @@
         </inertial>
     </link>
-    <joint name="${prefix}_mx28t_worm_joint" type="fixed">
+    <joint name="${prefix}_mx28t_worm_joint" type="revolute">
         <origin xyz="-0.00625 0.0112 0.0505" rpy="0 0 0"/>
+        <axis xyz="0 0 1" />
+        <limit lower="0" upper="-0.8" effort="10" velocity="10" />
         <parent link="${prefix}_mx28t_link"/>
         <child link="${prefix}_worm_link"/>
@@ -910,8 +912,11 @@
         </inertial>
     </link>
-    <joint name="${prefix}_gear1_shaft_joint" type="fixed">
+    <joint name="${prefix}_gear1_shaft_joint" type="revolute">
         <origin xyz="-0.00085 -0.000425 -0.0002" rpy="${PI/9} -${PI/18} ${PI/3}"/>
+        <axis xyz="0.64 -0.36 0" />
+        <limit lower="-0.8" upper="0" effort="10" velocity="10" />
         <parent link="${prefix}_gear1_shaft_link"/>
         <child link="${prefix}_gear1_link"/>
+        <mimic joint="${prefix}_mx28t_worm_joint" />
     </joint>
     <link name="${prefix}_gear2_link">
@@ -937,8 +942,11 @@
         </inertial>
     </link>
-    <joint name="${prefix}_gear2_shaft_joint" type="fixed">
+    <joint name="${prefix}_gear2_shaft_joint" type="revolute">
         <origin xyz="-0.00085 -0.000425 -0.0002" rpy="${PI/9} -${PI/18} ${PI/3}"/>
+        <axis xyz="0.64 -0.36 0" />
+        <limit lower="-0.8" upper="0" effort="10" velocity="10" />
         <parent link="${prefix}_gear2_shaft_link"/>
         <child link="${prefix}_gear2_link"/>
+        <mimic joint="${prefix}_mx28t_worm_joint" />
     </joint>
     <link name="${prefix}_gear3_link">
@@ -964,8 +972,11 @@
         </inertial>
     </link>
-    <joint name="${prefix}_gear3_shaft_joint" type="fixed">
+    <joint name="${prefix}_gear3_shaft_joint" type="revolute">
         <origin xyz="-0.00085 -0.000425 -0.0002" rpy="${PI/9} -${PI/18} ${PI/3}"/>
+        <axis xyz="0.64 -0.36 0" />
+        <limit lower="-0.8" upper="0" effort="10" velocity="10" />
         <parent link="${prefix}_gear3_shaft_link"/>
         <child link="${prefix}_gear3_link"/>
+        <mimic joint="${prefix}_mx28t_worm_joint" />
     </joint>
     <link name="${prefix}_gear1_shaft_retaining_ring1_link">

File: alaris_gripper_description/urdf/parts/finger.urdf.xacro (robot description, xacro)
@@ -2,4 +2,13 @@
 <robot name="alaris_gripper_finger" xmlns:xacro="http://www.ros.org/wiki/xacro">
 <xacro:macro name="alaris_gripper_finger" params="prefix finger_id parent *origin">
+    <link name="${prefix}_finger_${finger_id}_link1_revolution_point1"/>
+    <joint name="${prefix}_finger_${finger_id}_link1_revolution_point1_joint" type="revolute">
+        <xacro:insert_block name="origin"/>
+        <axis xyz="0.64 0.36 0" />
+        <limit lower="0" upper="-0.8" effort="10" velocity="10" />
+        <parent link="${parent}"/>
+        <child link="${prefix}_finger_${finger_id}_link1_revolution_point1"/>
+        <mimic joint="${prefix}_mx28t_worm_joint" />
+    </joint>
     <link name="${prefix}_finger_${finger_id}_link1_link">
         <visual>
@@ -25,6 +34,6 @@
     </link>
     <joint name="${prefix}_finger_${finger_id}_gear_link_joint" type="fixed">
-        <xacro:insert_block name="origin"/>
-        <parent link="${parent}"/>
+        <origin xyz="0.0012 -0.0025 -0.001" rpy="0 0 0"/>
+        <parent link="${prefix}_finger_${finger_id}_link1_revolution_point1"/>
         <child link="${prefix}_finger_${finger_id}_link1_link"/>
     </joint>

Commit message: Visually correct mechanical movement. Time for some simulation!

File: alaris_gripper_description/urdf/alaris_gripper.urdf.xacro (robot description, xacro)
@@ -9,11 +9,11 @@
     <xacro:alaris_gripper_base prefix="${prefix}"/>
     <xacro:alaris_gripper_finger prefix="${prefix}" finger_id="1" parent="${prefix}_palm_link">
-        <origin xyz="-0.0435 -0.00052 -0.006" rpy="0 0 -${2*PI/3}"/>
+        <origin xyz="-0.0435 -0.00052 -0.006" rpy="0 0 ${PI}"/>
     </xacro:alaris_gripper_finger>
     <xacro:alaris_gripper_finger prefix="${prefix}" finger_id="2" parent="${prefix}_palm_link">
-        <origin xyz="0.022 0.03785 -0.006" rpy="0 0 ${2*PI/3}"/>
+        <origin xyz="0.022 0.03785 -0.006" rpy="0 0 ${PI/3}"/>
     </xacro:alaris_gripper_finger>
     <xacro:alaris_gripper_finger prefix="${prefix}" finger_id="3" parent="${prefix}_palm_link">
-        <origin xyz="0.0226 -0.03785 -0.006" rpy="0 0 0"/>
+        <origin xyz="0.0226 -0.03785 -0.006" rpy="0 0 -${PI/3}"/>
     </xacro:alaris_gripper_finger>
 </robot>

File: alaris_gripper_description/urdf/parts/base.urdf.xacro (robot description, xacro)
@@ -157,5 +157,5 @@
         <origin xyz="-0.00625 0.0112 0.0505" rpy="0 0 0"/>
         <axis xyz="0 0 1" />
-        <limit lower="0" upper="-0.8" effort="10" velocity="10" />
+        <limit lower="-0.8" upper="0.8" effort="10" velocity="10" />
         <parent link="${prefix}_mx28t_link"/>
         <child link="${prefix}_worm_link"/>
@@ -915,5 +915,5 @@
         <origin xyz="-0.00085 -0.000425 -0.0002" rpy="${PI/9} -${PI/18} ${PI/3}"/>
         <axis xyz="-0.64 0.36 0" />
-        <limit lower="-0.8" upper="0" effort="10" velocity="10" />
+        <limit lower="-0.8" upper="0.8" effort="10" velocity="10" />
         <parent link="${prefix}_gear1_shaft_link"/>
         <child link="${prefix}_gear1_link"/>
@@ -945,5 +945,5 @@
         <origin xyz="-0.00085 -0.000425 -0.0002" rpy="${PI/9} -${PI/18} ${PI/3}"/>
         <axis xyz="0.64 -0.36 0" />
-        <limit lower="-0.8" upper="0" effort="10" velocity="10" />
+        <limit lower="-0.8" upper="0.8" effort="10" velocity="10" />
         <parent link="${prefix}_gear2_shaft_link"/>
         <child link="${prefix}_gear2_link"/>
@@ -975,5 +975,5 @@
         <origin xyz="-0.00085 -0.000425 -0.0002" rpy="${PI/9} -${PI/18} ${PI/3}"/>
         <axis xyz="-0.64 0.36 0" />
-        <limit lower="-0.8" upper="0" effort="10" velocity="10" />
+        <limit lower="-0.8" upper="0.8" effort="10" velocity="10" />
         <parent link="${prefix}_gear3_shaft_link"/>
         <child link="${prefix}_gear3_link"/>

File: alaris_gripper_description/urdf/parts/finger.urdf.xacro (robot description, xacro)
@@ -2,12 +2,41 @@
 <robot name="alaris_gripper_finger" xmlns:xacro="http://www.ros.org/wiki/xacro">
 <xacro:macro name="alaris_gripper_finger" params="prefix finger_id parent *origin">
+    <link name="${prefix}_finger_${finger_id}_bottom_shaft1_link">
+        <visual>
+            <origin xyz="0 0 0" rpy="0 0 0"/>
+            <geometry>
+                <mesh filename="package://alaris_gripper_description/meshes/Gripper_Assembly - shaft_3.STL" scale="0.001 0.001 0.001"/>
+            </geometry>
+            <material name="gray"/>
+        </visual>
+        <collision>
+            <origin xyz="0.0 0.0 0.0" rpy="0 0 0"/>
+            <geometry>
+                <mesh filename="package://alaris_gripper_description/meshes/Gripper_Assembly - shaft_3.STL" scale="0.001 0.001 0.001"/>
+            </geometry>
+        </collision>
+        <inertial>
+            <mass value="0.079" />
+            <origin xyz="0 0 0" />
+            <inertia ixx="0.003881243" ixy="0.0" ixz="0.0"
+                     iyy="0.000498940" iyz="0.0"
+                     izz="0.003879257" />
+        </inertial>
+    </link>
+    <joint name="${prefix}_finger_${finger_id}_link1_bottom_shaft1_joint" type="revolute">
+        <xacro:insert_block name="origin"/>
+        <axis xyz="0 1 0" />
+        <limit lower="-0.8" upper="0" effort="10" velocity="10" />
+        <parent link="${parent}"/>
+        <child link="${prefix}_finger_${finger_id}_bottom_shaft1_link"/>
+        <mimic joint="${prefix}_mx28t_worm_joint" multiplier="1"/>
+    </joint>
     <link name="${prefix}_finger_${finger_id}_link1_revolution_point1"/>
-    <joint name="${prefix}_finger_${finger_id}_link1_revolution_point1_joint" type="revolute">
-        <xacro:insert_block name="origin"/>
+    <joint name="${prefix}_finger_${finger_id}_link1_revolution_point1_joint" type="continuous">
+        <origin xyz="0 0 0" rpy="0 0 ${PI/3}"/>
         <axis xyz="0.64 0.36 0" />
-        <limit lower="0" upper="-0.8" effort="10" velocity="10" />
-        <parent link="${parent}"/>
+        <parent link="${prefix}_finger_${finger_id}_bottom_shaft1_link"/>
         <child link="${prefix}_finger_${finger_id}_link1_revolution_point1"/>
-        <mimic joint="${prefix}_mx28t_worm_joint" />
+        <mimic joint="${prefix}_finger_${finger_id}_phalanx2_revolution_point_joint" multiplier="0.49"/>
     </joint>
     <link name="${prefix}_finger_${finger_id}_link1_link">
@@ -38,4 +67,12 @@
         <child link="${prefix}_finger_${finger_id}_link1_link"/>
     </joint>
+    <link name="${prefix}_finger_${finger_id}_link1_revolution_point2"/>
+    <joint name="${prefix}_finger_${finger_id}_link1_revolution_point2_joint" type="continuous">
+        <origin xyz="0.01252 -0.0218 -0.0101" rpy="0 0 -${PI/3}"/>
+        <axis xyz="0 1 0" />
+        <parent link="${prefix}_finger_${finger_id}_link1_link"/>
+        <child link="${prefix}_finger_${finger_id}_link1_revolution_point2"/>
+        <mimic joint="${prefix}_finger_${finger_id}_phalanx2_revolution_point_joint" multiplier="-0.55"/>
+    </joint>
     <link name="${prefix}_finger_${finger_id}_link2_link">
         <visual>
@@ -61,6 +98,6 @@
     </link>
     <joint name="${prefix}_finger_${finger_id}_link1_link2_joint" type="fixed">
-        <origin xyz="0.01575 -0.0274 0.0239" rpy="0 0 0"/>
-        <parent link="${prefix}_finger_${finger_id}_link1_link"/>
+        <origin xyz="0.0065 0 0.034" rpy="0 0 ${PI/3}"/>
+        <parent link="${prefix}_finger_${finger_id}_link1_revolution_point2"/>
         <child link="${prefix}_finger_${finger_id}_link2_link"/>
     </joint>
@@ -88,8 +125,16 @@
     </link>
     <joint name="${prefix}_finger_${finger_id}_link1_phalanx1_joint" type="fixed">
-        <origin xyz="0.009 -0.01325 0.02" rpy="0 0 0"/>
-        <parent link="${prefix}_finger_${finger_id}_link1_link"/>
+        <origin xyz="0.01825 0.00075 0.01925" rpy="0 0 ${PI/3}"/>
+        <parent link="${prefix}_finger_${finger_id}_bottom_shaft1_link"/>
         <child link="${prefix}_finger_${finger_id}_phalanx1_link"/>
     </joint>
+    <link name="${prefix}_finger_${finger_id}_phalanx2_revolution_point"/>
+    <joint name="${prefix}_finger_${finger_id}_phalanx2_revolution_point_joint" type="revolute">
+        <origin xyz="0.004 -0.012 0.041" rpy="0 0 -${PI/3}"/>
+        <axis xyz="0 1 0" />
+        <limit lower="-0.8" upper="0" effort="10" velocity="10" />
+        <parent link="${prefix}_finger_${finger_id}_phalanx1_link"/>
+        <child link="${prefix}_finger_${finger_id}_phalanx2_revolution_point"/>
+    </joint>
     <link name="${prefix}_finger_${finger_id}_phalanx2_link">
         <visual>
@@ -115,6 +160,6 @@
     </link>
     <joint name="${prefix}_finger_${finger_id}_phalanx1_phalanx2_joint" type="fixed">
-        <origin xyz="0.0113 -0.022 0.057" rpy="0 0 0"/>
-        <parent link="${prefix}_finger_${finger_id}_phalanx1_link"/>
+        <origin xyz="0.013 0.001 0.016" rpy="0 0 ${PI/3}"/>
+        <parent link="${prefix}_finger_${finger_id}_phalanx2_revolution_point"/>
         <child link="${prefix}_finger_${finger_id}_phalanx2_link"/>
     </joint>
@@ -200,31 +245,4 @@
         <child link="${prefix}_finger_${finger_id}_top_shaft1_link"/>
     </joint>
-    <link name="${prefix}_finger_${finger_id}_bottom_shaft1_link">
-        <visual>
-            <origin xyz="0 0 0" rpy="0 0 0"/>
-            <geometry>
-                <mesh filename="package://alaris_gripper_description/meshes/Gripper_Assembly - shaft_3.STL" scale="0.001 0.001 0.001"/>
-            </geometry>
-            <material name="gray"/>
-        </visual>
-        <collision>
-            <origin xyz="0.0 0.0 0.0" rpy="0 0 0"/>
-            <geometry>
-                <mesh filename="package://alaris_gripper_description/meshes/Gripper_Assembly - shaft_3.STL" scale="0.001 0.001 0.001"/>
-            </geometry>
-        </collision>
-        <inertial>
-            <mass value="0.079" />
-            <origin xyz="0 0 0" />
-            <inertia ixx="0.003881243" ixy="0.0" ixz="0.0"
-                     iyy="0.000498940" iyz="0.0"
-                     izz="0.003879257" />
-        </inertial>
-    </link>
-    <joint name="${prefix}_finger_${finger_id}_link1_bottom_shaft1_joint" type="fixed">
-        <origin xyz="-0.00075 0.0025 0.001" rpy="0 0 -${PI/3}"/>
-        <parent link="${prefix}_finger_${finger_id}_link1_link"/>
-        <child link="${prefix}_finger_${finger_id}_bottom_shaft1_link"/>
-    </joint>
     <link name="${prefix}_finger_${finger_id}_bottom_shaft2_link">
         <visual>
