Commit message: Extra base details and new meshes path

File: alaris_gripper_description/urdf/parts/base.urdf.xacro (robot description, xacro)
@@ -2,19 +2,9 @@
 <robot name="alaris_gripper_base" xmlns:xacro="http://www.ros.org/wiki/xacro">
 <xacro:macro name="alaris_gripper_base" params="prefix">
-    <xacro:property name="PI" value="3.14159"/>
-    <material name="black">
-        <color rgba="0.2 0.2 0.2 1"/>
-    </material>
-    <material name="white">
-        <color rgba="1 1 1 1"/>
-    </material>
-    <material name="gray">
-        <color rgba="0.5 0.5 0.5 1"/>
-    </material>
     <link name="${prefix}_platform_link">
         <visual>
             <origin xyz="0 0 0" rpy="0 0 0"/>
             <geometry>
-                <mesh filename="package://alaris_gripper_description/meshes/fixed/Gripper_Assembly - platform.STL" scale="0.001 0.001 0.001"/>
+                <mesh filename="package://alaris_gripper_description/meshes/Gripper_Assembly - platform.STL" scale="0.001 0.001 0.001"/>
             </geometry>
             <material name="white"/>
@@ -23,5 +13,5 @@
             <origin xyz="0.0 0.0 0.0" rpy="0 0 0"/>
             <geometry>
-                <mesh filename="package://alaris_gripper_description/meshes/fixed/Gripper_Assembly - platform.STL" scale="0.001 0.001 0.001"/>
+                <mesh filename="package://alaris_gripper_description/meshes/Gripper_Assembly - platform.STL" scale="0.001 0.001 0.001"/>
             </geometry>
         </collision>
@@ -38,12 +28,12 @@
             <origin xyz="0 0 0" rpy="0 0 0"/>
             <geometry>
-                <mesh filename="package://alaris_gripper_description/meshes/fixed/Gripper_Assembly - MX28T.STL" scale="0.001 0.001 0.001"/>
-            </geometry>
-            <material name="black"/>
-        </visual>
-        <collision>
-            <origin xyz="0.0 0.0 0.0" rpy="0 0 0"/>
-            <geometry>
-                <mesh filename="package://alaris_gripper_description/meshes/fixed/Gripper_Assembly - MX28T.STL" scale="0.001 0.001 0.001"/>
+                <mesh filename="package://alaris_gripper_description/meshes/Gripper_Assembly - MX28T.STL" scale="0.001 0.001 0.001"/>
+            </geometry>
+            <material name="black"/>
+        </visual>
+        <collision>
+            <origin xyz="0.0 0.0 0.0" rpy="0 0 0"/>
+            <geometry>
+                <mesh filename="package://alaris_gripper_description/meshes/Gripper_Assembly - MX28T.STL" scale="0.001 0.001 0.001"/>
             </geometry>
         </collision>
@@ -65,12 +55,12 @@
             <origin xyz="0 0 0" rpy="0 0 0"/>
             <geometry>
-                <mesh filename="package://alaris_gripper_description/meshes/fixed/Gripper_Assembly - Standoff.STL" scale="0.001 0.001 0.001"/>
-            </geometry>
-            <material name="gray"/>
-        </visual>
-        <collision>
-            <origin xyz="0.0 0.0 0.0" rpy="0 0 0"/>
-            <geometry>
-                <mesh filename="package://alaris_gripper_description/meshes/fixed/Gripper_Assembly - Standoff.STL" scale="0.001 0.001 0.001"/>
+                <mesh filename="package://alaris_gripper_description/meshes/Gripper_Assembly - Standoff.STL" scale="0.001 0.001 0.001"/>
+            </geometry>
+            <material name="gray"/>
+        </visual>
+        <collision>
+            <origin xyz="0.0 0.0 0.0" rpy="0 0 0"/>
+            <geometry>
+                <mesh filename="package://alaris_gripper_description/meshes/Gripper_Assembly - Standoff.STL" scale="0.001 0.001 0.001"/>
             </geometry>
         </collision>
@@ -92,12 +82,12 @@
             <origin xyz="0 0 0" rpy="0 0 0"/>
             <geometry>
-                <mesh filename="package://alaris_gripper_description/meshes/fixed/Gripper_Assembly - Standoff.STL" scale="0.001 0.001 0.001"/>
-            </geometry>
-            <material name="gray"/>
-        </visual>
-        <collision>
-            <origin xyz="0.0 0.0 0.0" rpy="0 0 0"/>
-            <geometry>
-                <mesh filename="package://alaris_gripper_description/meshes/fixed/Gripper_Assembly - Standoff.STL" scale="0.001 0.001 0.001"/>
+                <mesh filename="package://alaris_gripper_description/meshes/Gripper_Assembly - Standoff.STL" scale="0.001 0.001 0.001"/>
+            </geometry>
+            <material name="gray"/>
+        </visual>
+        <collision>
+            <origin xyz="0.0 0.0 0.0" rpy="0 0 0"/>
+            <geometry>
+                <mesh filename="package://alaris_gripper_description/meshes/Gripper_Assembly - Standoff.STL" scale="0.001 0.001 0.001"/>
             </geometry>
         </collision>
@@ -119,12 +109,12 @@
             <origin xyz="0 0 0" rpy="0 0 0"/>
             <geometry>
-                <mesh filename="package://alaris_gripper_description/meshes/fixed/Gripper_Assembly - Standoff.STL" scale="0.001 0.001 0.001"/>
-            </geometry>
-            <material name="gray"/>
-        </visual>
-        <collision>
-            <origin xyz="0.0 0.0 0.0" rpy="0 0 0"/>
-            <geometry>
-                <mesh filename="package://alaris_gripper_description/meshes/fixed/Gripper_Assembly - Standoff.STL" scale="0.001 0.001 0.001"/>
+                <mesh filename="package://alaris_gripper_description/meshes/Gripper_Assembly - Standoff.STL" scale="0.001 0.001 0.001"/>
+            </geometry>
+            <material name="gray"/>
+        </visual>
+        <collision>
+            <origin xyz="0.0 0.0 0.0" rpy="0 0 0"/>
+            <geometry>
+                <mesh filename="package://alaris_gripper_description/meshes/Gripper_Assembly - Standoff.STL" scale="0.001 0.001 0.001"/>
             </geometry>
         </collision>
@@ -146,5 +136,5 @@
             <origin xyz="0 0 0" rpy="0 0 0"/>
             <geometry>
-                <mesh filename="package://alaris_gripper_description/meshes/fixed/Gripper_Assembly - worm.STL" scale="0.001 0.001 0.001"/>
+                <mesh filename="package://alaris_gripper_description/meshes/Gripper_Assembly - worm.STL" scale="0.001 0.001 0.001"/>
             </geometry>
             <material name="white"/>
@@ -153,5 +143,5 @@
             <origin xyz="0.0 0.0 0.0" rpy="0 0 0"/>
             <geometry>
-                <mesh filename="package://alaris_gripper_description/meshes/fixed/Gripper_Assembly - worm.STL" scale="0.001 0.001 0.001"/>
+                <mesh filename="package://alaris_gripper_description/meshes/Gripper_Assembly - worm.STL" scale="0.001 0.001 0.001"/>
             </geometry>
         </collision>
@@ -173,5 +163,5 @@
             <origin xyz="0 0 0" rpy="0 0 0"/>
             <geometry>
-                <mesh filename="package://alaris_gripper_description/meshes/fixed/Gripper_Assembly - palm.STL" scale="0.001 0.001 0.001"/>
+                <mesh filename="package://alaris_gripper_description/meshes/Gripper_Assembly - palm.STL" scale="0.001 0.001 0.001"/>
             </geometry>
             <material name="white"/>
@@ -180,5 +170,5 @@
             <origin xyz="0.0 0.0 0.0" rpy="0 0 0"/>
             <geometry>
-                <mesh filename="package://alaris_gripper_description/meshes/fixed/Gripper_Assembly - palm.STL" scale="0.001 0.001 0.001"/>
+                <mesh filename="package://alaris_gripper_description/meshes/Gripper_Assembly - palm.STL" scale="0.001 0.001 0.001"/>
             </geometry>
         </collision>
@@ -200,12 +190,12 @@
             <origin xyz="0 0 0" rpy="0 0 0"/>
             <geometry>
-                <mesh filename="package://alaris_gripper_description/meshes/fixed/Gripper_Assembly - screw_standoff.STL" scale="0.001 0.001 0.001"/>
-            </geometry>
-            <material name="black"/>
-        </visual>
-        <collision>
-            <origin xyz="0.0 0.0 0.0" rpy="0 0 0"/>
-            <geometry>
-                <mesh filename="package://alaris_gripper_description/meshes/fixed/Gripper_Assembly - screw_standoff.STL" scale="0.001 0.001 0.001"/>
+                <mesh filename="package://alaris_gripper_description/meshes/Gripper_Assembly - screw_standoff.STL" scale="0.001 0.001 0.001"/>
+            </geometry>
+            <material name="black"/>
+        </visual>
+        <collision>
+            <origin xyz="0.0 0.0 0.0" rpy="0 0 0"/>
+            <geometry>
+                <mesh filename="package://alaris_gripper_description/meshes/Gripper_Assembly - screw_standoff.STL" scale="0.001 0.001 0.001"/>
             </geometry>
         </collision>
@@ -227,12 +217,12 @@
             <origin xyz="0 0 0" rpy="0 0 0"/>
             <geometry>
-                <mesh filename="package://alaris_gripper_description/meshes/fixed/Gripper_Assembly - screw_standoff.STL" scale="0.001 0.001 0.001"/>
-            </geometry>
-            <material name="black"/>
-        </visual>
-        <collision>
-            <origin xyz="0.0 0.0 0.0" rpy="0 0 0"/>
-            <geometry>
-                <mesh filename="package://alaris_gripper_description/meshes/fixed/Gripper_Assembly - screw_standoff.STL" scale="0.001 0.001 0.001"/>
+                <mesh filename="package://alaris_gripper_description/meshes/Gripper_Assembly - screw_standoff.STL" scale="0.001 0.001 0.001"/>
+            </geometry>
+            <material name="black"/>
+        </visual>
+        <collision>
+            <origin xyz="0.0 0.0 0.0" rpy="0 0 0"/>
+            <geometry>
+                <mesh filename="package://alaris_gripper_description/meshes/Gripper_Assembly - screw_standoff.STL" scale="0.001 0.001 0.001"/>
             </geometry>
         </collision>
@@ -254,12 +244,12 @@
             <origin xyz="0 0 0" rpy="0 0 0"/>
             <geometry>
-                <mesh filename="package://alaris_gripper_description/meshes/fixed/Gripper_Assembly - screw_standoff.STL" scale="0.001 0.001 0.001"/>
-            </geometry>
-            <material name="black"/>
-        </visual>
-        <collision>
-            <origin xyz="0.0 0.0 0.0" rpy="0 0 0"/>
-            <geometry>
-                <mesh filename="package://alaris_gripper_description/meshes/fixed/Gripper_Assembly - screw_standoff.STL" scale="0.001 0.001 0.001"/>
+                <mesh filename="package://alaris_gripper_description/meshes/Gripper_Assembly - screw_standoff.STL" scale="0.001 0.001 0.001"/>
+            </geometry>
+            <material name="black"/>
+        </visual>
+        <collision>
+            <origin xyz="0.0 0.0 0.0" rpy="0 0 0"/>
+            <geometry>
+                <mesh filename="package://alaris_gripper_description/meshes/Gripper_Assembly - screw_standoff.STL" scale="0.001 0.001 0.001"/>
             </geometry>
         </collision>
@@ -281,12 +271,12 @@
             <origin xyz="0 0 0" rpy="0 0 0"/>
             <geometry>
-                <mesh filename="package://alaris_gripper_description/meshes/fixed/Gripper_Assembly - screw_standoff.STL" scale="0.001 0.001 0.001"/>
-            </geometry>
-            <material name="black"/>
-        </visual>
-        <collision>
-            <origin xyz="0.0 0.0 0.0" rpy="0 0 0"/>
-            <geometry>
-                <mesh filename="package://alaris_gripper_description/meshes/fixed/Gripper_Assembly - screw_standoff.STL" scale="0.001 0.001 0.001"/>
+                <mesh filename="package://alaris_gripper_description/meshes/Gripper_Assembly - screw_standoff.STL" scale="0.001 0.001 0.001"/>
+            </geometry>
+            <material name="black"/>
+        </visual>
+        <collision>
+            <origin xyz="0.0 0.0 0.0" rpy="0 0 0"/>
+            <geometry>
+                <mesh filename="package://alaris_gripper_description/meshes/Gripper_Assembly - screw_standoff.STL" scale="0.001 0.001 0.001"/>
             </geometry>
         </collision>
@@ -308,12 +298,12 @@
             <origin xyz="0 0 0" rpy="0 0 0"/>
             <geometry>
-                <mesh filename="package://alaris_gripper_description/meshes/fixed/Gripper_Assembly - screw_standoff.STL" scale="0.001 0.001 0.001"/>
-            </geometry>
-            <material name="black"/>
-        </visual>
-        <collision>
-            <origin xyz="0.0 0.0 0.0" rpy="0 0 0"/>
-            <geometry>
-                <mesh filename="package://alaris_gripper_description/meshes/fixed/Gripper_Assembly - screw_standoff.STL" scale="0.001 0.001 0.001"/>
+                <mesh filename="package://alaris_gripper_description/meshes/Gripper_Assembly - screw_standoff.STL" scale="0.001 0.001 0.001"/>
+            </geometry>
+            <material name="black"/>
+        </visual>
+        <collision>
+            <origin xyz="0.0 0.0 0.0" rpy="0 0 0"/>
+            <geometry>
+                <mesh filename="package://alaris_gripper_description/meshes/Gripper_Assembly - screw_standoff.STL" scale="0.001 0.001 0.001"/>
             </geometry>
         </collision>
@@ -335,12 +325,12 @@
             <origin xyz="0 0 0" rpy="0 0 0"/>
             <geometry>
-                <mesh filename="package://alaris_gripper_description/meshes/fixed/Gripper_Assembly - screw_standoff.STL" scale="0.001 0.001 0.001"/>
-            </geometry>
-            <material name="black"/>
-        </visual>
-        <collision>
-            <origin xyz="0.0 0.0 0.0" rpy="0 0 0"/>
-            <geometry>
-                <mesh filename="package://alaris_gripper_description/meshes/fixed/Gripper_Assembly - screw_standoff.STL" scale="0.001 0.001 0.001"/>
+                <mesh filename="package://alaris_gripper_description/meshes/Gripper_Assembly - screw_standoff.STL" scale="0.001 0.001 0.001"/>
+            </geometry>
+            <material name="black"/>
+        </visual>
+        <collision>
+            <origin xyz="0.0 0.0 0.0" rpy="0 0 0"/>
+            <geometry>
+                <mesh filename="package://alaris_gripper_description/meshes/Gripper_Assembly - screw_standoff.STL" scale="0.001 0.001 0.001"/>
             </geometry>
         </collision>
@@ -362,12 +352,12 @@
             <origin xyz="0 0 0" rpy="0 0 0"/>
             <geometry>
-                <mesh filename="package://alaris_gripper_description/meshes/fixed/Gripper_Assembly - rubber_palm.STL" scale="0.001 0.001 0.001"/>
-            </geometry>
-            <material name="black"/>
-        </visual>
-        <collision>
-            <origin xyz="0.0 0.0 0.0" rpy="0 0 0"/>
-            <geometry>
-                <mesh filename="package://alaris_gripper_description/meshes/fixed/Gripper_Assembly - rubber_palm.STL" scale="0.001 0.001 0.001"/>
+                <mesh filename="package://alaris_gripper_description/meshes/Gripper_Assembly - rubber_palm.STL" scale="0.001 0.001 0.001"/>
+            </geometry>
+            <material name="black"/>
+        </visual>
+        <collision>
+            <origin xyz="0.0 0.0 0.0" rpy="0 0 0"/>
+            <geometry>
+                <mesh filename="package://alaris_gripper_description/meshes/Gripper_Assembly - rubber_palm.STL" scale="0.001 0.001 0.001"/>
             </geometry>
         </collision>
@@ -389,12 +379,12 @@
             <origin xyz="0 0 0" rpy="0 0 0"/>
             <geometry>
-                <mesh filename="package://alaris_gripper_description/meshes/fixed/Gripper_Assembly - M2.5_Screw_for_platform.STL" scale="0.001 0.001 0.001"/>
-            </geometry>
-            <material name="black"/>
-        </visual>
-        <collision>
-            <origin xyz="0.0 0.0 0.0" rpy="0 0 0"/>
-            <geometry>
-                <mesh filename="package://alaris_gripper_description/meshes/fixed/Gripper_Assembly - M2.5_Screw_for_platform.STL" scale="0.001 0.001 0.001"/>
+                <mesh filename="package://alaris_gripper_description/meshes/Gripper_Assembly - M2.5_Screw_for_platform.STL" scale="0.001 0.001 0.001"/>
+            </geometry>
+            <material name="black"/>
+        </visual>
+        <collision>
+            <origin xyz="0.0 0.0 0.0" rpy="0 0 0"/>
+            <geometry>
+                <mesh filename="package://alaris_gripper_description/meshes/Gripper_Assembly - M2.5_Screw_for_platform.STL" scale="0.001 0.001 0.001"/>
             </geometry>
         </collision>
@@ -416,12 +406,12 @@
             <origin xyz="0 0 0" rpy="0 0 0"/>
             <geometry>
-                <mesh filename="package://alaris_gripper_description/meshes/fixed/Gripper_Assembly - M2.5_Screw_for_platform.STL" scale="0.001 0.001 0.001"/>
-            </geometry>
-            <material name="black"/>
-        </visual>
-        <collision>
-            <origin xyz="0.0 0.0 0.0" rpy="0 0 0"/>
-            <geometry>
-                <mesh filename="package://alaris_gripper_description/meshes/fixed/Gripper_Assembly - M2.5_Screw_for_platform.STL" scale="0.001 0.001 0.001"/>
+                <mesh filename="package://alaris_gripper_description/meshes/Gripper_Assembly - M2.5_Screw_for_platform.STL" scale="0.001 0.001 0.001"/>
+            </geometry>
+            <material name="black"/>
+        </visual>
+        <collision>
+            <origin xyz="0.0 0.0 0.0" rpy="0 0 0"/>
+            <geometry>
+                <mesh filename="package://alaris_gripper_description/meshes/Gripper_Assembly - M2.5_Screw_for_platform.STL" scale="0.001 0.001 0.001"/>
             </geometry>
         </collision>
@@ -443,12 +433,12 @@
             <origin xyz="0 0 0" rpy="0 0 0"/>
             <geometry>
-                <mesh filename="package://alaris_gripper_description/meshes/fixed/Gripper_Assembly - M2.5_Screw_for_platform.STL" scale="0.001 0.001 0.001"/>
-            </geometry>
-            <material name="black"/>
-        </visual>
-        <collision>
-            <origin xyz="0.0 0.0 0.0" rpy="0 0 0"/>
-            <geometry>
-                <mesh filename="package://alaris_gripper_description/meshes/fixed/Gripper_Assembly - M2.5_Screw_for_platform.STL" scale="0.001 0.001 0.001"/>
+                <mesh filename="package://alaris_gripper_description/meshes/Gripper_Assembly - M2.5_Screw_for_platform.STL" scale="0.001 0.001 0.001"/>
+            </geometry>
+            <material name="black"/>
+        </visual>
+        <collision>
+            <origin xyz="0.0 0.0 0.0" rpy="0 0 0"/>
+            <geometry>
+                <mesh filename="package://alaris_gripper_description/meshes/Gripper_Assembly - M2.5_Screw_for_platform.STL" scale="0.001 0.001 0.001"/>
             </geometry>
         </collision>
@@ -470,12 +460,12 @@
             <origin xyz="0 0 0" rpy="0 0 0"/>
             <geometry>
-                <mesh filename="package://alaris_gripper_description/meshes/fixed/Gripper_Assembly - M2.5_Screw_for_platform.STL" scale="0.001 0.001 0.001"/>
-            </geometry>
-            <material name="black"/>
-        </visual>
-        <collision>
-            <origin xyz="0.0 0.0 0.0" rpy="0 0 0"/>
-            <geometry>
-                <mesh filename="package://alaris_gripper_description/meshes/fixed/Gripper_Assembly - M2.5_Screw_for_platform.STL" scale="0.001 0.001 0.001"/>
+                <mesh filename="package://alaris_gripper_description/meshes/Gripper_Assembly - M2.5_Screw_for_platform.STL" scale="0.001 0.001 0.001"/>
+            </geometry>
+            <material name="black"/>
+        </visual>
+        <collision>
+            <origin xyz="0.0 0.0 0.0" rpy="0 0 0"/>
+            <geometry>
+                <mesh filename="package://alaris_gripper_description/meshes/Gripper_Assembly - M2.5_Screw_for_platform.STL" scale="0.001 0.001 0.001"/>
             </geometry>
         </collision>
@@ -497,12 +487,12 @@
             <origin xyz="0 0 0" rpy="0 0 0"/>
             <geometry>
-                <mesh filename="package://alaris_gripper_description/meshes/fixed/Gripper_Assembly - M2.5_Screw_for_platform.STL" scale="0.001 0.001 0.001"/>
-            </geometry>
-            <material name="black"/>
-        </visual>
-        <collision>
-            <origin xyz="0.0 0.0 0.0" rpy="0 0 0"/>
-            <geometry>
-                <mesh filename="package://alaris_gripper_description/meshes/fixed/Gripper_Assembly - M2.5_Screw_for_platform.STL" scale="0.001 0.001 0.001"/>
+                <mesh filename="package://alaris_gripper_description/meshes/Gripper_Assembly - M2.5_Screw_for_platform.STL" scale="0.001 0.001 0.001"/>
+            </geometry>
+            <material name="black"/>
+        </visual>
+        <collision>
+            <origin xyz="0.0 0.0 0.0" rpy="0 0 0"/>
+            <geometry>
+                <mesh filename="package://alaris_gripper_description/meshes/Gripper_Assembly - M2.5_Screw_for_platform.STL" scale="0.001 0.001 0.001"/>
             </geometry>
         </collision>
@@ -524,12 +514,12 @@
             <origin xyz="0 0 0" rpy="0 0 0"/>
             <geometry>
-                <mesh filename="package://alaris_gripper_description/meshes/fixed/Gripper_Assembly - M2.5_Screw_for_platform.STL" scale="0.001 0.001 0.001"/>
-            </geometry>
-            <material name="black"/>
-        </visual>
-        <collision>
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
Commit message: Fixed gear rotation for better visual effect

File: alaris_gripper_description/urdf/parts/base.urdf.xacro (robot description, xacro)
@@ -914,5 +914,5 @@
     <joint name="${prefix}_gear1_shaft_joint" type="revolute">
         <origin xyz="-0.00085 -0.000425 -0.0002" rpy="${PI/9} -${PI/18} ${PI/3}"/>
-        <axis xyz="0.64 -0.36 0" />
+        <axis xyz="-0.64 0.36 0" />
         <limit lower="-0.8" upper="0" effort="10" velocity="10" />
         <parent link="${prefix}_gear1_shaft_link"/>
@@ -974,5 +974,5 @@
     <joint name="${prefix}_gear3_shaft_joint" type="revolute">
         <origin xyz="-0.00085 -0.000425 -0.0002" rpy="${PI/9} -${PI/18} ${PI/3}"/>
-        <axis xyz="0.64 -0.36 0" />
+        <axis xyz="-0.64 0.36 0" />
         <limit lower="-0.8" upper="0" effort="10" velocity="10" />
         <parent link="${prefix}_gear3_shaft_link"/>
