Commit message: Changes towards Gazebo simulation. It now needs correct masses and inertia

File: alaris_gripper_description/urdf/parts/base.urdf.xacro (robot description, xacro)
@@ -160,4 +160,5 @@
         <parent link="${prefix}_mx28t_link"/>
         <child link="${prefix}_worm_link"/>
+        <dynamics damping="0.02" friction="0.0" />
     </joint>
     <link name="${prefix}_palm_link">
@@ -919,4 +920,5 @@
         <child link="${prefix}_gear1_link"/>
         <mimic joint="${prefix}_mx28t_worm_joint" />
+        <dynamics damping="0.02" friction="0.0" />
     </joint>
     <link name="${prefix}_gear2_link">
@@ -949,4 +951,5 @@
         <child link="${prefix}_gear2_link"/>
         <mimic joint="${prefix}_mx28t_worm_joint" />
+        <dynamics damping="0.02" friction="0.0" />
     </joint>
     <link name="${prefix}_gear3_link">
@@ -979,4 +982,5 @@
         <child link="${prefix}_gear3_link"/>
         <mimic joint="${prefix}_mx28t_worm_joint" />
+        <dynamics damping="0.02" friction="0.0" />
     </joint>
     <link name="${prefix}_gear1_shaft_retaining_ring1_link">
@@ -991,5 +995,5 @@
             <origin xyz="0.0 0.0 0.0" rpy="0 0 0"/>
             <geometry>
-                <mesh filename="package://alaris_gripper_description/meshes/Gripper_Assembly - Retaining ring_2" scale="0.001 0.001 0.001"/>
+                <mesh filename="package://alaris_gripper_description/meshes/Gripper_Assembly - Retaining ring_2.STL" scale="0.001 0.001 0.001"/>
             </geometry>
         </collision>
@@ -1018,5 +1022,5 @@
             <origin xyz="0.0 0.0 0.0" rpy="0 0 0"/>
             <geometry>
-                <mesh filename="package://alaris_gripper_description/meshes/Gripper_Assembly - Retaining ring_2" scale="0.001 0.001 0.001"/>
+                <mesh filename="package://alaris_gripper_description/meshes/Gripper_Assembly - Retaining ring_2.STL" scale="0.001 0.001 0.001"/>
             </geometry>
         </collision>
@@ -1045,5 +1049,5 @@
             <origin xyz="0.0 0.0 0.0" rpy="0 0 0"/>
             <geometry>
-                <mesh filename="package://alaris_gripper_description/meshes/Gripper_Assembly - Retaining ring_2" scale="0.001 0.001 0.001"/>
+                <mesh filename="package://alaris_gripper_description/meshes/Gripper_Assembly - Retaining ring_2.STL" scale="0.001 0.001 0.001"/>
             </geometry>
         </collision>
@@ -1072,5 +1076,5 @@
             <origin xyz="0.0 0.0 0.0" rpy="0 0 0"/>
             <geometry>
-                <mesh filename="package://alaris_gripper_description/meshes/Gripper_Assembly - Retaining ring_2" scale="0.001 0.001 0.001"/>
+                <mesh filename="package://alaris_gripper_description/meshes/Gripper_Assembly - Retaining ring_2.STL" scale="0.001 0.001 0.001"/>
             </geometry>
         </collision>
@@ -1099,5 +1103,5 @@
             <origin xyz="0.0 0.0 0.0" rpy="0 0 0"/>
             <geometry>
-                <mesh filename="package://alaris_gripper_description/meshes/Gripper_Assembly - Retaining ring_2" scale="0.001 0.001 0.001"/>
+                <mesh filename="package://alaris_gripper_description/meshes/Gripper_Assembly - Retaining ring_2.STL" scale="0.001 0.001 0.001"/>
             </geometry>
         </collision>
@@ -1126,5 +1130,5 @@
             <origin xyz="0.0 0.0 0.0" rpy="0 0 0"/>
             <geometry>
-                <mesh filename="package://alaris_gripper_description/meshes/Gripper_Assembly - Retaining ring_2" scale="0.001 0.001 0.001"/>
+                <mesh filename="package://alaris_gripper_description/meshes/Gripper_Assembly - Retaining ring_2.STL" scale="0.001 0.001 0.001"/>
             </geometry>
         </collision>
@@ -1142,4 +1146,175 @@
         <child link="${prefix}_gear3_shaft_retaining_ring2_link"/>
     </joint>
+    <!-- Gazebo Related -->
+     <gazebo>
+        <plugin name="gazebo_ros_control" filename="libgazebo_ros_control.so">
+          <robotNamespace>/</robotNamespace>
+        </plugin>
+        <plugin name="${prefix}_gear1_shaft_joint_plugin" filename="libroboticsgroup_gazebo_mimic_joint_plugin.so">
+        <joint>${prefix}_mx28t_worm_joint</joint>
+        <mimicJoint>${prefix}_gear1_shaft_joint</mimicJoint>
+        <multiplier>1</multiplier>
+        <offset>0</offset>
+        <sensitiveness>0</sensitiveness>   <!-- if absolute difference between setpoint and process value is below this threshold, do nothing; 0.0 = disable [rad] -->
+        <maxEffort>10</maxEffort> <!-- only taken into account if has_pid:=true [Nm] -->
+        <robotNamespace>/</robotNamespace>
+      </plugin>
+        <plugin name="${prefix}_gear2_shaft_joint_plugin" filename="libroboticsgroup_gazebo_mimic_joint_plugin.so">
+        <joint>${prefix}_mx28t_worm_joint</joint>
+        <mimicJoint>${prefix}_gear2_shaft_joint</mimicJoint>
+        <multiplier>1</multiplier>
+        <offset>0</offset>
+        <sensitiveness>0</sensitiveness>   <!-- if absolute difference between setpoint and process value is below this threshold, do nothing; 0.0 = disable [rad] -->
+        <maxEffort>10</maxEffort> <!-- only taken into account if has_pid:=true [Nm] -->
+        <robotNamespace>/</robotNamespace>
+      </plugin>
+        <plugin name="${prefix}_gear3_shaft_joint_plugin" filename="libroboticsgroup_gazebo_mimic_joint_plugin.so">
+        <joint>${prefix}_mx28t_worm_joint</joint>
+        <mimicJoint>${prefix}_gear3_shaft_joint</mimicJoint>
+        <multiplier>1</multiplier>
+        <offset>0</offset>
+        <sensitiveness>0</sensitiveness>   <!-- if absolute difference between setpoint and process value is below this threshold, do nothing; 0.0 = disable [rad] -->
+        <maxEffort>10</maxEffort> <!-- only taken into account if has_pid:=true [Nm] -->
+        <robotNamespace>/</robotNamespace>
+      </plugin>
+    </gazebo>
+    <gazebo reference="${prefix}_gear3_shaft_link">
+      <self_collide>false</self_collide>
+    </gazebo>
+    <gazebo reference="${prefix}_platform_link">
+      <self_collide>false</self_collide>
+    </gazebo>
+    <gazebo reference="${prefix}_mx28t_link">
+      <self_collide>false</self_collide>
+    </gazebo>
+    <gazebo reference="${prefix}_standoff1_link">
+      <self_collide>false</self_collide>
+    </gazebo>
+    <gazebo reference="${prefix}_standoff2_link">
+      <self_collide>false</self_collide>
+    </gazebo>
+    <gazebo reference="${prefix}_standoff3_link">
+      <self_collide>false</self_collide>
+    </gazebo>
+    <gazebo reference="${prefix}_worm_link">
+      <self_collide>false</self_collide>
+    </gazebo>
+    <gazebo reference="${prefix}_palm_link">
+      <self_collide>false</self_collide>
+    </gazebo>
+    <gazebo reference="${prefix}_standoff1_screw1_link">
+      <self_collide>false</self_collide>
+    </gazebo>
+    <gazebo reference="${prefix}_standoff2_screw1_link">
+      <self_collide>false</self_collide>
+    </gazebo>
+    <gazebo reference="${prefix}_standoff3_screw1_link">
+      <self_collide>false</self_collide>
+    </gazebo>
+    <gazebo reference="${prefix}_standoff1_screw2_link">
+      <self_collide>false</self_collide>
+    </gazebo>
+    <gazebo reference="${prefix}_standoff2_screw2_link">
+      <self_collide>false</self_collide>
+    </gazebo>
+    <gazebo reference="${prefix}_standoff3_screw2_link">
+      <self_collide>false</self_collide>
+    </gazebo>
+    <gazebo reference="${prefix}_palm_rubber_link">
+      <self_collide>false</self_collide>
+    </gazebo>
+    <gazebo reference="${prefix}_mx28t_screw1_link">
+      <self_collide>false</self_collide>
+    </gazebo>
+    <gazebo reference="${prefix}_mx28t_screw2_link">
+      <self_collide>false</self_collide>
+    </gazebo>
+    <gazebo reference="${prefix}_mx28t_screw3_link">
+      <self_collide>false</self_collide>
+    </gazebo>
+    <gazebo reference="${prefix}_mx28t_screw4_link">
+      <self_collide>false</self_collide>
+    </gazebo>
+    <gazebo reference="${prefix}_mx28t_screw5_link">
+      <self_collide>false</self_collide>
+    </gazebo>
+    <gazebo reference="${prefix}_mx28t_screw6_link">
+      <self_collide>false</self_collide>
+    </gazebo>
+    <gazebo reference="${prefix}_mx28t_screw7_link">
+      <self_collide>false</self_collide>
+    </gazebo>
+    <gazebo reference="${prefix}_mx28t_screw8_link">
+      <self_collide>false</self_collide>
+    </gazebo>
+    <gazebo reference="${prefix}_mx28t_nut1_link">
+      <self_collide>false</self_collide>
+    </gazebo>
+    <gazebo reference="${prefix}_mx28t_nut2_link">
+      <self_collide>false</self_collide>
+    </gazebo>
+    <gazebo reference="${prefix}_mx28t_nut3_link">
+      <self_collide>false</self_collide>
+    </gazebo>
+    <gazebo reference="${prefix}_mx28t_nut4_link">
+      <self_collide>false</self_collide>
+    </gazebo>
+    <gazebo reference="${prefix}_mx28t_nut5_link">
+      <self_collide>false</self_collide>
+    </gazebo>
+    <gazebo reference="${prefix}_mx28t_nut6_link">
+      <self_collide>false</self_collide>
+    </gazebo>
+    <gazebo reference="${prefix}_mx28t_nut7_link">
+      <self_collide>false</self_collide>
+    </gazebo>
+    <gazebo reference="${prefix}_mx28t_nut8_link">
+      <self_collide>false</self_collide>
+    </gazebo>
+    <gazebo reference="${prefix}_gear1_shaft_link">
+      <self_collide>false</self_collide>
+    </gazebo>
+    <gazebo reference="${prefix}_gear2_shaft_link">
+      <self_collide>false</self_collide>
+    </gazebo>
+    <gazebo reference="${prefix}_gear3_shaft_link">
+      <self_collide>false</self_collide>
+    </gazebo>
+    <gazebo reference="${prefix}_gear1_link">
+      <self_collide>false</self_collide>
+    </gazebo>
+    <gazebo reference="${prefix}_gear2_link">
+      <self_collide>false</self_collide>
+    </gazebo>
+    <gazebo reference="${prefix}_gear3_link">
+      <self_collide>false</self_collide>
+    </gazebo>
+    <gazebo reference="${prefix}_gear1_shaft_retaining_ring1_link">
+      <self_collide>false</self_collide>
+    </gazebo>
+    <gazebo reference="${prefix}_gear1_shaft_retaining_ring2_link">
+      <self_collide>false</self_collide>
+    </gazebo>
+    <gazebo reference="${prefix}_gear2_shaft_retaining_ring1_link">
+      <self_collide>false</self_collide>
+    </gazebo>
+    <gazebo reference="${prefix}_gear2_shaft_retaining_ring2_link">
+      <self_collide>false</self_collide>
+    </gazebo>
+    <gazebo reference="${prefix}_gear3_shaft_retaining_ring1_link">
+      <self_collide>false</self_collide>
+    </gazebo>
+    <gazebo reference="${prefix}_gear3_shaft_retaining_ring2_link">
+      <self_collide>false</self_collide>
+    </gazebo>
+    <transmission name="${prefix}_mx28t_worm_trans" type="SimpleTransmission">
+        <type>transmission_interface/SimpleTransmission</type>
+        <actuator name="${prefix}_mx28t_worm_joint_motor">
+            <mechanicalReduction>1</mechanicalReduction>
+        </actuator>
+        <joint name="${prefix}_mx28t_worm_joint">
+            <hardwareInterface>hardware_interface/EffortJointInterface</hardwareInterface>
+        </joint>
+    </transmission>
 </xacro:macro>
 </robot>

File: alaris_gripper_description/urdf/parts/finger.urdf.xacro (robot description, xacro)
@@ -31,4 +31,5 @@
         <child link="${prefix}_finger_${finger_id}_bottom_shaft1_link"/>
         <mimic joint="${prefix}_mx28t_worm_joint" multiplier="1"/>
+        <dynamics damping="0.02" friction="0.0" />
     </joint>
     <link name="${prefix}_finger_${finger_id}_link1_revolution_point1"/>
@@ -39,4 +40,5 @@
         <child link="${prefix}_finger_${finger_id}_link1_revolution_point1"/>
         <mimic joint="${prefix}_finger_${finger_id}_phalanx2_revolution_point_joint" multiplier="0.49"/>
+        <dynamics damping="0.02" friction="0.0" />
     </joint>
     <link name="${prefix}_finger_${finger_id}_link1_link">
@@ -136,4 +138,5 @@
         <parent link="${prefix}_finger_${finger_id}_phalanx1_link"/>
         <child link="${prefix}_finger_${finger_id}_phalanx2_revolution_point"/>
+        <dynamics damping="0.02" friction="0.0" />
     </joint>
     <link name="${prefix}_finger_${finger_id}_phalanx2_link">
@@ -299,4 +302,85 @@
         <child link="${prefix}_finger_${finger_id}_top_shaft2_link"/>
     </joint>
+    <!-- Gazebo Related -->
+     <gazebo>
+        <plugin name="gazebo_ros_control" filename="libgazebo_ros_control.so">
+          <robotNamespace>/</robotNamespace>
+        </plugin>
+        <plugin name="${prefix}_finger_${finger_id}_link1_bottom_shaft1_joint_plugin" filename="libroboticsgroup_gazebo_mimic_joint_plugin.so">
+        <joint>${prefix}_mx28t_worm_joint</joint>
+        <mimicJoint>${prefix}_finger_${finger_id}_link1_bottom_shaft1_joint</mimicJoint>
+        <multiplier>1</multiplier>
+        <offset>0</offset>
+        <sensitiveness>0</sensitiveness>   <!-- if absolute difference between setpoint and process value is below this threshold, do nothing; 0.0 = disable [rad] -->
+        <maxEffort>10</maxEffort> <!-- only taken into account if has_pid:=true [Nm] -->
+        <robotNamespace>/</robotNamespace>
+      </plugin>
+        <plugin name="${prefix}_finger_${finger_id}_link1_revolution_point1_joint_plugin" filename="libroboticsgroup_gazebo_mimic_joint_plugin.so">
+        <joint>${prefix}_finger_${finger_id}_phalanx2_revolution_point_joint</joint>
+        <mimicJoint>${prefix}_finger_${finger_id}_link1_revolution_point1_joint</mimicJoint>
+        <multiplier>0.49</multiplier>
+        <offset>0</offset>
+        <sensitiveness>0</sensitiveness>   <!-- if absolute difference between setpoint and process value is below this threshold, do nothing; 0.0 = disable [rad] -->
+        <maxEffort>10</maxEffort> <!-- only taken into account if has_pid:=true [Nm] -->
+        <robotNamespace>/</robotNamespace>
+      </plugin>
+        <plugin name="${prefix}_finger_${finger_id}_link1_revolution_point2_joint_plugin" filename="libroboticsgroup_gazebo_mimic_joint_plugin.so">
+        <joint>${prefix}_finger_${finger_id}_phalanx2_revolution_point_joint</joint>
+        <mimicJoint>${prefix}_finger_${finger_id}_link1_revolution_point2_joint</mimicJoint>
+        <multiplier>-0.55</multiplier>
+        <offset>0</offset>
+        <sensitiveness>0</sensitiveness>   <!-- if absolute difference between setpoint and process value is below this threshold, do nothing; 0.0 = disable [rad] -->
+        <maxEffort>10</maxEffort> <!-- only taken into account if has_pid:=true [Nm] -->
+        <robotNamespace>/</robotNamespace>
+      </plugin>
+    </gazebo>
+    <transmission name="${prefix}_finger_${finger_id}_phalanx2_revolution_point_trans" type="SimpleTransmission">
+        <type>transmission_interface/SimpleTransmission</type>
+        <actuator name="${prefix}_finger_${finger_id}_phalanx2_revolution_point_motor">
+            <mechanicalReduction>1</mechanicalReduction>
+        </actuator>
+        <joint name="${prefix}_finger_${finger_id}_phalanx2_revolution_point_joint">
+            <hardwareInterface>hardware_interface/EffortJointInterface</hardwareInterface>
+        </joint>
+    </transmission>
+    <gazebo reference="${prefix}_finger_${finger_id}_bottom_shaft1_link">
+      <self_collide>false</self_collide>
+    </gazebo>
+    <gazebo reference="${prefix}_finger_${finger_id}_link1_revolution_point1">
+      <self_collide>false</self_collide>
+    </gazebo>
+    <gazebo reference="${prefix}_finger_${finger_id}_link1_link">
+      <self_collide>false</self_collide>
+    </gazebo>
+    <gazebo reference="${prefix}_finger_${finger_id}_link1_revolution_point2">
+      <self_collide>false</self_collide>
+    </gazebo>
+    <gazebo reference="${prefix}_finger_${finger_id}_link2_link">
+      <self_collide>false</self_collide>
+    </gazebo>
+    <gazebo reference="${prefix}_finger_${finger_id}_phalanx1_link">
+      <self_collide>false</self_collide>
+    </gazebo>
+    <gazebo reference="${prefix}_finger_${finger_id}_phalanx2_revolution_point">
+      <self_collide>false</self_collide>
+    </gazebo>
+    <gazebo reference="${prefix}_finger_${finger_id}_phalanx2_link">
+      <self_collide>false</self_collide>
+    </gazebo>
+    <gazebo reference="${prefix}_finger_${finger_id}_rubber_phalanx1_link">
+      <self_collide>false</self_collide>
+    </gazebo>
+    <gazebo reference="${prefix}_finger_${finger_id}_rubber_phalanx2_link">
+      <self_collide>false</self_collide>
+    </gazebo>
+    <gazebo reference="${prefix}_finger_${finger_id}_top_shaft1_link">
+      <self_collide>false</self_collide>
+    </gazebo>
+    <gazebo reference="${prefix}_finger_${finger_id}_bottom_shaft2_link">
+      <self_collide>false</self_collide>
+    </gazebo>
+    <gazebo reference="${prefix}_finger_${finger_id}_top_shaft2_link">
+      <self_collide>false</self_collide>
+    </gazebo>
 </xacro:macro>
 </robot>
