Commit message: Changes towards better gripper simulation

File: alaris_gripper_description/urdf/parts/base.urdf.xacro (robot description, xacro)
@@ -1,6 +1,9 @@
 <?xml version="1.0"?>
 <robot name="alaris_gripper_base" xmlns:xacro="http://www.ros.org/wiki/xacro">
+<!-- TODO: Accurate inertia and CoM -->
+<!-- TODO2: Contact coefficients -->
 <xacro:macro name="alaris_gripper_base" params="prefix">
     <link name="${prefix}_platform_link">
+        <static>true</static>
         <visual>
             <origin xyz="0 0 0" rpy="0 0 0"/>
@@ -14,34 +17,33 @@
             <geometry>
                 <mesh filename="package://alaris_gripper_description/meshes/Gripper_Assembly - platform.STL" scale="0.001 0.001 0.001"/>
+            </geometry>
+        </collision>
+        <!-- <inertial>
+            <mass value="0.03" />
+            <origin xyz="0 0 0" />
+           <inertia  ixx="0.0251360610696" ixy="0" ixz="0" iyy="0.0251415862243" iyz="0" izz="0.0499576469124" />
+        </inertial> -->
+    </link>
+    <link name="${prefix}_mx28t_link">
+        <visual>
+            <origin xyz="0 0 0" rpy="0 0 0"/>
+            <geometry>
+                <mesh filename="package://alaris_gripper_description/meshes/Gripper_Assembly - MX28T.STL" scale="0.001 0.001 0.001"/>
+            </geometry>
+            <material name="black"/>
+        </visual>
+        <collision>
+            <origin xyz="0.0 0.0 0.0" rpy="0 0 0"/>
+            <geometry>
+                <mesh filename="package://alaris_gripper_description/meshes/Gripper_Assembly - MX28T.STL" scale="0.001 0.001 0.001"/>
             </geometry>
         </collision>
         <inertial>
-            <mass value="0.2" />
-            <origin xyz="0 0 0" />
-            <inertia ixx="0.003881243" ixy="0.0" ixz="0.0"
-                     iyy="0.000498940" iyz="0.0"
-                     izz="0.003879257" />
-        </inertial>
-    </link>
-    <link name="${prefix}_mx28t_link">
-        <visual>
-            <origin xyz="0 0 0" rpy="0 0 0"/>
-            <geometry>
-                <mesh filename="package://alaris_gripper_description/meshes/Gripper_Assembly - MX28T.STL" scale="0.001 0.001 0.001"/>
-            </geometry>
-            <material name="black"/>
-        </visual>
-        <collision>
-            <origin xyz="0.0 0.0 0.0" rpy="0 0 0"/>
-            <geometry>
-                <mesh filename="package://alaris_gripper_description/meshes/Gripper_Assembly - MX28T.STL" scale="0.001 0.001 0.001"/>
-            </geometry>
-        </collision>
-        <inertial>
-            <mass value="0.079" />
-            <origin xyz="0 0 0" />
-            <inertia ixx="0.003881243" ixy="0.0" ixz="0.0"
-                     iyy="0.000498940" iyz="0.0"
-                     izz="0.003879257" />
+            <mass value="2.079" />
+            <!-- TODO -->
+            <!-- Real mass here is 0.079, but adding 2kg increases stability. -->
+            <!-- <mass value="0.079" /> -->
+            <origin xyz="0 0 0" />
+           <inertia  ixx="0.0348708168255" ixy="0" ixz="0" iyy="0.0303839715998" iyz="0" izz="0.0375755319567" />
         </inertial>
     </link>
@@ -65,11 +67,9 @@
             </geometry>
         </collision>
-        <inertial>
-            <mass value="0.5" />
-            <origin xyz="0 0 0" />
-            <inertia ixx="0.003881243" ixy="0.0" ixz="0.0"
-                     iyy="0.000498940" iyz="0.0"
-                     izz="0.003879257" />
-        </inertial>
+        <!-- <inertial>
+            <mass value="0.005" />
+            <origin xyz="0 0 0" />
+           <inertia  ixx="0.00243615089784" ixy="0" ixz="0" iyy="0.00244175112182" iyz="0" izz="3.9202407236e-05" />
+        </inertial> -->
     </link>
     <joint name="${prefix}_platform_standoff1_joint" type="fixed">
@@ -92,11 +92,9 @@
             </geometry>
         </collision>
-        <inertial>
-            <mass value="0.5" />
-            <origin xyz="0 0 0" />
-            <inertia ixx="0.003881243" ixy="0.0" ixz="0.0"
-                     iyy="0.000498940" iyz="0.0"
-                     izz="0.003879257" />
-        </inertial>
+        <!-- <inertial>
+            <mass value="0.005" />
+            <origin xyz="0 0 0" />
+           <inertia  ixx="0.00243615089784" ixy="0" ixz="0" iyy="0.00244175112182" iyz="0" izz="3.9202407236e-05" />
+        </inertial> -->
     </link>
     <joint name="${prefix}_platform_standoff2_joint" type="fixed">
@@ -119,11 +117,9 @@
             </geometry>
         </collision>
-        <inertial>
-            <mass value="0.5" />
-            <origin xyz="0 0 0" />
-            <inertia ixx="0.003881243" ixy="0.0" ixz="0.0"
-                     iyy="0.000498940" iyz="0.0"
-                     izz="0.003879257" />
-        </inertial>
+        <!-- <inertial>
+            <mass value="0.005" />
+            <origin xyz="0 0 0" />
+           <inertia  ixx="0.00243615089784" ixy="0" ixz="0" iyy="0.00244175112182" iyz="0" izz="3.9202407236e-05" />
+        </inertial> -->
     </link>
     <joint name="${prefix}_platform_standoff3_joint" type="fixed">
@@ -140,16 +136,14 @@
             <material name="white"/>
         </visual>
-        <collision>
+        <!-- <collision>
             <origin xyz="0.0 0.0 0.0" rpy="0 0 0"/>
             <geometry>
                 <mesh filename="package://alaris_gripper_description/meshes/Gripper_Assembly - worm.STL" scale="0.001 0.001 0.001"/>
             </geometry>
-        </collision>
+        </collision> -->
         <inertial>
-            <mass value="0.5" />
-            <origin xyz="0 0 0" />
-            <inertia ixx="0.003881243" ixy="0.0" ixz="0.0"
-                     iyy="0.000498940" iyz="0.0"
-                     izz="0.003879257" />
+            <mass value="0.015" />
+            <origin xyz="0 0 0" />
+           <inertia  ixx="0.30427083939" ixy="0" ixz="0" iyy="0.304272499683" iyz="0" izz="0.12454325515" />
         </inertial>
     </link>
@@ -176,11 +170,9 @@
             </geometry>
         </collision>
-        <inertial>
-            <mass value="0.5" />
-            <origin xyz="0 0 0" />
-            <inertia ixx="0.003881243" ixy="0.0" ixz="0.0"
-                     iyy="0.000498940" iyz="0.0"
-                     izz="0.003879257" />
-        </inertial>
+        <!-- <inertial>
+            <mass value="0.03" />
+            <origin xyz="0 0 0" />
+           <inertia  ixx="0.0273707858005" ixy="0" ixz="0" iyy="0.0277986279135" iyz="0" izz="0.0475711129826" />
+        </inertial> -->
     </link>
     <joint name="${prefix}_platform_palm_joint" type="fixed">
@@ -197,17 +189,15 @@
             <material name="black"/>
         </visual>
-        <collision>
+        <!-- <collision>
             <origin xyz="0.0 0.0 0.0" rpy="0 0 0"/>
             <geometry>
                 <mesh filename="package://alaris_gripper_description/meshes/Gripper_Assembly - screw_standoff.STL" scale="0.001 0.001 0.001"/>
             </geometry>
-        </collision>
-        <inertial>
-            <mass value="0.5" />
-            <origin xyz="0 0 0" />
-            <inertia ixx="0.003881243" ixy="0.0" ixz="0.0"
-                     iyy="0.000498940" iyz="0.0"
-                     izz="0.003879257" />
-        </inertial>
+        </collision> -->
+        <!-- <inertial>
+            <mass value="0.001" />
+            <origin xyz="0 0 0" />
+           <inertia  ixx="2.12724885605e-05" ixy="0" ixz="0" iyy="2.12724969418e-05" iyz="0" izz="7.24086635252e-06" />
+        </inertial> -->
     </link>
     <joint name="${prefix}_standoff1_screw1_joint" type="fixed">
@@ -224,17 +214,15 @@
             <material name="black"/>
         </visual>
-        <collision>
+        <!-- <collision>
             <origin xyz="0.0 0.0 0.0" rpy="0 0 0"/>
             <geometry>
                 <mesh filename="package://alaris_gripper_description/meshes/Gripper_Assembly - screw_standoff.STL" scale="0.001 0.001 0.001"/>
             </geometry>
-        </collision>
-        <inertial>
-            <mass value="0.5" />
-            <origin xyz="0 0 0" />
-            <inertia ixx="0.003881243" ixy="0.0" ixz="0.0"
-                     iyy="0.000498940" iyz="0.0"
-                     izz="0.003879257" />
-        </inertial>
+        </collision> -->
+        <!-- <inertial>
+            <mass value="0.001" />
+            <origin xyz="0 0 0" />
+           <inertia  ixx="2.12724885605e-05" ixy="0" ixz="0" iyy="2.12724969418e-05" iyz="0" izz="7.24086635252e-06" />
+        </inertial> -->
     </link>
     <joint name="${prefix}_standoff2_screw1_joint" type="fixed">
@@ -251,17 +239,15 @@
             <material name="black"/>
         </visual>
-        <collision>
+        <!-- <collision>
             <origin xyz="0.0 0.0 0.0" rpy="0 0 0"/>
             <geometry>
                 <mesh filename="package://alaris_gripper_description/meshes/Gripper_Assembly - screw_standoff.STL" scale="0.001 0.001 0.001"/>
             </geometry>
-        </collision>
-        <inertial>
-            <mass value="0.5" />
-            <origin xyz="0 0 0" />
-            <inertia ixx="0.003881243" ixy="0.0" ixz="0.0"
-                     iyy="0.000498940" iyz="0.0"
-                     izz="0.003879257" />
-        </inertial>
+        </collision> -->
+        <!-- <inertial>
+            <mass value="0.001" />
+            <origin xyz="0 0 0" />
+           <inertia  ixx="2.12724885605e-05" ixy="0" ixz="0" iyy="2.12724969418e-05" iyz="0" izz="7.24086635252e-06" />
+        </inertial> -->
     </link>
     <joint name="${prefix}_standoff3_screw1_joint" type="fixed">
@@ -278,17 +264,15 @@
             <material name="black"/>
         </visual>
-        <collision>
+        <!-- <collision>
             <origin xyz="0.0 0.0 0.0" rpy="0 0 0"/>
             <geometry>
                 <mesh filename="package://alaris_gripper_description/meshes/Gripper_Assembly - screw_standoff.STL" scale="0.001 0.001 0.001"/>
             </geometry>
-        </collision>
-        <inertial>
-            <mass value="0.5" />
-            <origin xyz="0 0 0" />
-            <inertia ixx="0.003881243" ixy="0.0" ixz="0.0"
-                     iyy="0.000498940" iyz="0.0"
-                     izz="0.003879257" />
-        </inertial>
+        </collision> -->
+        <!-- <inertial>
+            <mass value="0.001" />
+            <origin xyz="0 0 0" />
+           <inertia  ixx="2.12724885605e-05" ixy="0" ixz="0" iyy="2.12724969418e-05" iyz="0" izz="7.24086635252e-06" />
+        </inertial> -->
     </link>
     <joint name="${prefix}_standoff1_screw2_joint" type="fixed">
@@ -305,17 +289,15 @@
             <material name="black"/>
         </visual>
-        <collision>
+        <!-- <collision>
             <origin xyz="0.0 0.0 0.0" rpy="0 0 0"/>
             <geometry>
                 <mesh filename="package://alaris_gripper_description/meshes/Gripper_Assembly - screw_standoff.STL" scale="0.001 0.001 0.001"/>
             </geometry>
-        </collision>
-        <inertial>
-            <mass value="0.5" />
-            <origin xyz="0 0 0" />
-            <inertia ixx="0.003881243" ixy="0.0" ixz="0.0"
-                     iyy="0.000498940" iyz="0.0"
-                     izz="0.003879257" />
-        </inertial>
+        </collision> -->
+        <!-- <inertial>
+            <mass value="0.001" />
+            <origin xyz="0 0 0" />
+           <inertia  ixx="2.12724885605e-05" ixy="0" ixz="0" iyy="2.12724969418e-05" iyz="0" izz="7.24086635252e-06" />
+        </inertial> -->
     </link>
     <joint name="${prefix}_standoff2_screw2_joint" type="fixed">
@@ -332,17 +314,15 @@
             <material name="black"/>
         </visual>
-        <collision>
+        <!-- <collision>
             <origin xyz="0.0 0.0 0.0" rpy="0 0 0"/>
             <geometry>
                 <mesh filename="package://alaris_gripper_description/meshes/Gripper_Assembly - screw_standoff.STL" scale="0.001 0.001 0.001"/>
             </geometry>
-        </collision>
-        <inertial>
-            <mass value="0.5" />
-            <origin xyz="0 0 0" />
-            <inertia ixx="0.003881243" ixy="0.0" ixz="0.0"
-                     iyy="0.000498940" iyz="0.0"
-                     izz="0.003879257" />
-        </inertial>
+        </collision> -->
+        <!-- <inertial>
+            <mass value="0.001" />
+            <origin xyz="0 0 0" />
+           <inertia  ixx="2.12724885605e-05" ixy="0" ixz="0" iyy="2.12724969418e-05" iyz="0" izz="7.24086635252e-06" />
+        </inertial> -->
     </link>
     <joint name="${prefix}_standoff3_screw2_joint" type="fixed">
@@ -359,17 +339,15 @@
             <material name="black"/>
         </visual>
-        <collision>
+        <!-- <collision>
             <origin xyz="0.0 0.0 0.0" rpy="0 0 0"/>
             <geometry>
                 <mesh filename="package://alaris_gripper_description/meshes/Gripper_Assembly - rubber_palm.STL" scale="0.001 0.001 0.001"/>
             </geometry>
-        </collision>
-        <inertial>
-            <mass value="0.5" />
-            <origin xyz="0 0 0" />
-            <inertia ixx="0.003881243" ixy="0.0" ixz="0.0"
-                     iyy="0.000498940" iyz="0.0"
-                     izz="0.003879257" />
-        </inertial>
+        </collision> -->
+        <!-- <inertial>
+            <mass value="0.003" />
+            <origin xyz="0 0 0" />
+           <inertia  ixx="0.00207151182299" ixy="0" ixz="0" iyy="0.00176457324947" iyz="0" izz="0.00383158506173" />
+        </inertial> -->
     </link>
     <joint name="${prefix}_palm_rubber_joint" type="fixed">
@@ -386,17 +364,15 @@
             <material name="black"/>
         </visual>
-        <collision>
-            <origin xyz="0.0 0.0 0.0" rpy="0 0 0"/>
-            <geometry>
-                <mesh filename="package://alaris_gripper_description/meshes/Gripper_Assembly - M2.5_Screw_for_platform.STL" scale="0.001 0.001 0.001"/>
-            </geometry>
-        </collision>
-        <inertial>
-            <mass value="0.5" />
-            <origin xyz="0 0 0" />
-            <inertia ixx="0.003881243" ixy="0.0" ixz="0.0"
-                     iyy="0.000498940" iyz="0.0"
-                     izz="0.003879257" />
-        </inertial>
+        <!-- <collision>
+            <origin xyz="0.0 0.0 0.0" rpy="0 0 0"/>
+            <geometry>
+                <mesh filename="package://alaris_gripper_description/meshes/Gripper_Assembly - M2.5_Screw_for_platform.STL" scale="0.001 0.001 0.001"/>
+            </geometry>
+        </collision> -->
+        <!-- <inertial>
+            <mass value="0.001" />
+            <origin xyz="0 0 0" />
+           <inertia  ixx="1.46989051635e-05" ixy="0" ixz="0" iyy="1.47083333333e-05" iyz="0" izz="3.36557183013e-06" />
+        </inertial> -->
     </link>
     <joint name="${prefix}_mx28t_screw1_joint" type="fixed">
@@ -413,17 +389,15 @@
             <material name="black"/>
         </visual>
-        <collision>
-            <origin xyz="0.0 0.0 0.0" rpy="0 0 0"/>
-            <geometry>
-                <mesh filename="package://alaris_gripper_description/meshes/Gripper_Assembly - M2.5_Screw_for_platform.STL" scale="0.001 0.001 0.001"/>
-            </geometry>
-        </collision>
-        <inertial>
-            <mass value="0.5" />
-            <origin xyz="0 0 0" />
-            <inertia ixx="0.003881243" ixy="0.0" ixz="0.0"
-                     iyy="0.000498940" iyz="0.0"
-                     izz="0.003879257" />
-        </inertial>
+        <!-- <collision>
+            <origin xyz="0.0 0.0 0.0" rpy="0 0 0"/>
+            <geometry>
+                <mesh filename="package://alaris_gripper_description/meshes/Gripper_Assembly - M2.5_Screw_for_platform.STL" scale="0.001 0.001 0.001"/>
+            </geometry>
+        </collision> -->
+        <!-- <inertial>
+            <mass value="0.001" />
+            <origin xyz="0 0 0" />
+           <inertia  ixx="1.46989051635e-05" ixy="0" ixz="0" iyy="1.47083333333e-05" iyz="0" izz="3.36557183013e-06" />
+        </inertial> -->
     </link>
     <joint name="${prefix}_mx28t_screw2_joint" type="fixed">
@@ -440,17 +414,15 @@
             <material name="black"/>
         </visual>
-        <collision>
-            <origin xyz="0.0 0.0 0.0" rpy="0 0 0"/>
-            <geometry>
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